Commit message: adding apf planner

File: src/my_bot/description/actual_camera_corr_rect_obj.xacro (robot description, xacro)
@@ -5,5 +5,5 @@
             <parent link="${prefix}chassis"/>
             <child link="${prefix}camera_link"/>
-            <origin xyz="0.28 0 0.20" rpy="0 0 0"/>
+            <origin xyz="0.23 0 0.20" rpy="0 0 0"/>
         </joint>
         <link name="${prefix}camera_link">

File: src/my_bot/description/actual_depth_camera_corr_rect_obj.xacro (robot description, xacro)
@@ -5,5 +5,5 @@
             <parent link="${prefix}chassis"/>
             <child link="${prefix}depth_camera_link"/>
-            <origin xyz="0.28 0 0.20" rpy="0 0 0"/>
+            <origin xyz="0.23 0 0.20" rpy="0 0 0"/>
         </joint>
         <link name="${prefix}depth_camera_link">

File: src/my_bot/description/actual_lidar_corr_rect_obj.xacro (robot description, xacro)
@@ -6,5 +6,5 @@
             <parent link="${prefix}chassis"/>
             <child link="${prefix}laser_frame"/>
-            <origin xyz="0.28 0 0.20" rpy="0 0 0"/>
+            <origin xyz="0.23 0 0.20" rpy="0 0 0"/>
         </joint>
         <link name="${prefix}laser_frame">

File: src/my_bot/description/actual_robot_rect_obj_core_corr.xacro (robot description, xacro)
@@ -39,5 +39,5 @@
             <origin xyz="0 0 0.08" />
             <geometry>
-                <box size="0.6 0.6 0.16"/>
+                <box size="0.5 0.5 0.16"/>
             </geometry>
             <material name="white" />
@@ -46,8 +46,8 @@
             <origin xyz="0 0 0.08" />
             <geometry>
-                <box size="0.6 0.6 0.16"/>
+                <box size="0.5 0.5 0.16"/>
             </geometry>
         </collision>
-        <xacro:inertial_box mass="1.0" x="0.6" y="0.6" z="0.16">
+        <xacro:inertial_box mass="1.0" x="0.5" y="0.5" z="0.16">
             <origin xyz="0 0 0.08" rpy="0 0 0"/>
         </xacro:inertial_box>

File: src/my_bot/description/actual_robot_rect_obj_corr.urdf.xacro (robot description, xacro)
@@ -6,9 +6,9 @@
     <xacro:include filename="actual_camera_corr_rect_obj.xacro"/>
     <xacro:include filename="actual_depth_camera_corr_rect_obj.xacro"/>
-    <!--xacro:include filename="actual_imu_corr_rect_obj.xacro"/-->
+    <xacro:include filename="actual_imu_corr_rect_obj.xacro"/>
     <xacro:rect_obj prefix=""/>
     <xacro:lidar_module prefix=""/>
     <xacro:camera_module prefix=""/>
     <xacro:depth_camera_module prefix=""/>
-    <!--xacro:imu_module prefix=""/-->
+    <xacro:imu_module prefix=""/>
 </robot>
